Commit message: Changed the xacro fails to avoid repetition

File: ca_description/urdf/sensors/cliff_sensors.xacro (robot description, xacro)
@@ -5,41 +5,28 @@
   <xacro:include filename="$(find ca_description)/urdf/sensors/cliff_sensors_gazebo.xacro"/>
   <xacro:property name="parent_link" value="base_link"/>
-  <xacro:property name="name_side_left" value="side_left"/>
-  <xacro:property name="name_side_right" value="side_right"/>
-  <xacro:property name="name_front_left" value="front_left"/>
-  <xacro:property name="name_front_right" value="front_right"/>
-  <joint name="${name_side_left}_cliff_sensor_joint" type="fixed">
+  <xacro:macro name="cliff_links_joints" params="name *origin">
+    <joint name="${name}_cliff_sensor_joint" type="fixed">
+      <xacro:insert_block name='origin' />
+      <parent link="${parent_link}" />
+      <child link="${name}_cliff_sensor_link" />
+    </joint>
+    <link name="${name}_cliff_sensor_link" />
+  </xacro:macro>
+  <xacro:cliff_links_joints name="side_left">
     <origin xyz="0.07 0.14 0.01" rpy="0 ${pi/2} 0" />
-    <parent link="${parent_link}" />
-    <child link="${name_side_left}_cliff_sensor_link" />
-  </joint>
-  <joint name="${name_side_right}_cliff_sensor_joint" type="fixed">
+  </xacro:cliff_links_joints>
+  <xacro:cliff_links_joints name="side_right">
     <origin xyz="0.07 -0.14 0.01" rpy="0 ${pi/2} 0" />
-    <parent link="${parent_link}" />
-    <child link="${name_side_right}_cliff_sensor_link" />
-  </joint>
-  <joint name="${name_front_left}_front_cliff_sensor_joint" type="fixed">
+  </xacro:cliff_links_joints>
+  <xacro:cliff_links_joints name="front_left">
     <origin xyz="0.15 0.04 0.01" rpy="0 ${pi/2} 0" />
-    <parent link="${parent_link}" />
-    <child link="${name_front_left}_cliff_sensor_link" />
-  </joint>
-  <joint name="${name_front_right}_cliff_sensor_joint" type="fixed">
+  </xacro:cliff_links_joints>
+  <xacro:cliff_links_joints name="front_right">
     <origin xyz="0.15 -0.04 0.01" rpy="0 ${pi/2} 0" />
-    <parent link="${parent_link}" />
-    <child link="${name_front_right}_cliff_sensor_link" />
-  </joint>
-  <link name="${name_side_left}_cliff_sensor_link">
-    <xacro:dummy_inertia/>
-  </link>
-  <link name="${name_side_right}_cliff_sensor_link">
-    <xacro:dummy_inertia/>
-  </link>
-  <link name="${name_front_left}_cliff_sensor_link">
-    <xacro:dummy_inertia/>
-  </link>
-  <link name="${name_front_right}_cliff_sensor_link">
-    <xacro:dummy_inertia/>
-  </link>
-  <xacro:sim_create_cliff_sensors visualize="${visualize}"/>
+  </xacro:cliff_links_joints>
+  <xacro:sim_create_cliff_sensors visualize="${visualize}" name="side_left"/>
+  <xacro:sim_create_cliff_sensors visualize="${visualize}" name="side_right"/>
+  <xacro:sim_create_cliff_sensors visualize="${visualize}" name="front_left"/>
+  <xacro:sim_create_cliff_sensors visualize="${visualize}" name="front_right"/>
 </xacro:macro>
 </robot>

File: ca_description/urdf/sensors/cliff_sensors_gazebo.xacro (robot description, xacro)
@@ -1,10 +1,9 @@
 <?xml version="1.0" ?>
 <robot xmlns:xacro="http://ros.org/wiki/xacro">
-<xacro:macro name="sim_create_cliff_sensors" params="visualize:=false">
+<xacro:macro name="sim_create_cliff_sensors" params="visualize:=false name">
   <xacro:property name="min_range_m" value="0.01"/>
   <xacro:property name="max_range_m" value="0.04"/>
   <xacro:property name="rate_hz" value="20.0"/>
   <xacro:property name="min_cliff_value_cm" value="3.5"/>
-  <xacro:macro name="gazebo_cliff_sensor" params="name">
     <gazebo reference="${name}_cliff_sensor_link">
       <sensor type="ray" name="${name}_cliff_sensor">
@@ -35,9 +34,4 @@
       </sensor>
     </gazebo>
-  </xacro:macro>
-  <xacro:gazebo_cliff_sensor name="${name_side_left}"/>
-  <xacro:gazebo_cliff_sensor name="${name_side_right}"/>
-  <xacro:gazebo_cliff_sensor name="${name_front_left}"/>
-  <xacro:gazebo_cliff_sensor name="${name_front_right}"/>
 </xacro:macro>
 </robot>

Commit message: Addressed the xacro comments

File: ca_description/urdf/sensors/cliff_sensors.xacro (robot description, xacro)
@@ -5,28 +5,25 @@
   <xacro:include filename="$(find ca_description)/urdf/sensors/cliff_sensors_gazebo.xacro"/>
   <xacro:property name="parent_link" value="base_link"/>
-  <xacro:macro name="cliff_links_joints" params="name *origin">
+  <xacro:macro name="cliff" params="name *origin">
     <joint name="${name}_cliff_sensor_joint" type="fixed">
-      <xacro:insert_block name='origin' />
+      <xacro:insert_block name="origin" />
       <parent link="${parent_link}" />
       <child link="${name}_cliff_sensor_link" />
     </joint>
     <link name="${name}_cliff_sensor_link" />
+    <xacro:cliff_plugin visualize="${visualize}" name="${name}"/>
   </xacro:macro>
-  <xacro:cliff_links_joints name="side_left">
-    <origin xyz="0.07 0.14 0.01" rpy="0 ${pi/2} 0" />
-  </xacro:cliff_links_joints>
-  <xacro:cliff_links_joints name="side_right">
-    <origin xyz="0.07 -0.14 0.01" rpy="0 ${pi/2} 0" />
-  </xacro:cliff_links_joints>
-  <xacro:cliff_links_joints name="front_left">
-    <origin xyz="0.15 0.04 0.01" rpy="0 ${pi/2} 0" />
-  </xacro:cliff_links_joints>
-  <xacro:cliff_links_joints name="front_right">
-    <origin xyz="0.15 -0.04 0.01" rpy="0 ${pi/2} 0" />
-  </xacro:cliff_links_joints>
-  <xacro:sim_create_cliff_sensors visualize="${visualize}" name="side_left"/>
-  <xacro:sim_create_cliff_sensors visualize="${visualize}" name="side_right"/>
-  <xacro:sim_create_cliff_sensors visualize="${visualize}" name="front_left"/>
-  <xacro:sim_create_cliff_sensors visualize="${visualize}" name="front_right"/>
+  <xacro:cliff name="side_left">
+    <origin xyz="0.07 0.14 0.01" rpy="0 ${pi/2 - 0.09} 0" />
+  </xacro:cliff>
+  <xacro:cliff name="side_right">
+    <origin xyz="0.07 -0.14 0.01" rpy="0 ${pi/2 - 0.09} 0" />
+  </xacro:cliff>
+  <xacro:cliff name="front_left">
+    <origin xyz="0.15 0.04 0.01" rpy="0 ${pi/2 - 0.09} 0" />
+  </xacro:cliff>
+  <xacro:cliff name="front_right">
+    <origin xyz="0.15 -0.04 0.01" rpy="0 ${pi/2 - 0.09} 0" />
+  </xacro:cliff>
 </xacro:macro>
 </robot>

File: ca_description/urdf/sensors/cliff_sensors_gazebo.xacro (robot description, xacro)
@@ -1,9 +1,9 @@
 <?xml version="1.0" ?>
 <robot xmlns:xacro="http://ros.org/wiki/xacro">
-<xacro:macro name="sim_create_cliff_sensors" params="visualize:=false name">
+<xacro:macro name="cliff_plugin" params="visualize:=false name">
   <xacro:property name="min_range_m" value="0.01"/>
   <xacro:property name="max_range_m" value="0.04"/>
   <xacro:property name="rate_hz" value="20.0"/>
-  <xacro:property name="min_cliff_value_cm" value="3.5"/>
+  <xacro:property name="min_cliff_value_cm" value="3.85"/>
     <gazebo reference="${name}_cliff_sensor_link">
       <sensor type="ray" name="${name}_cliff_sensor">
