Commit message: Added functional cliff msg publisher

File: ca_description/urdf/create_2.xacro (robot description, xacro)
@@ -3,4 +3,6 @@
   <xacro:include filename="$(find ca_description)/urdf/create_base.xacro"/>
   <xacro:include filename="$(find ca_description)/urdf/roomblock.xacro"/>
+  <xacro:arg name="robot_number" default="1"/>
+  <xacro:property name="robot_number" value="$(arg robot_number)"/>
   <xacro:property name="wheel_separation" value="0.235"/>
   <xacro:property name="base_diameter" value="0.3485"/>

File: ca_description/urdf/create_base_gazebo.xacro (robot description, xacro)
@@ -77,4 +77,12 @@
       <material>Gazebo/Grey</material>
     </gazebo>
+    <!-- Cliff Publisher detector -->
+    <gazebo>
+      <plugin name="cliff_msg_publisher" filename="libcliff_msg_publisher.so">
+        <updateRate>10</updateRate>
+        <robotNumber>${robot_number}</robotNumber>
+        <frameName>/base_link</frameName>
+      </plugin>
+    </gazebo>
   </xacro:macro>
 </robot>

Commit message: Addressed most of the comments

File: ca_description/urdf/create_2.xacro (robot description, xacro)
@@ -3,6 +3,5 @@
   <xacro:include filename="$(find ca_description)/urdf/create_base.xacro"/>
   <xacro:include filename="$(find ca_description)/urdf/roomblock.xacro"/>
-  <xacro:arg name="robot_number" default="1"/>
-  <xacro:property name="robot_number" value="$(arg robot_number)"/>
+  <xacro:property name="robot_name" value="$(arg robot_name)"/>
   <xacro:property name="wheel_separation" value="0.235"/>
   <xacro:property name="base_diameter" value="0.3485"/>

File: ca_description/urdf/create_base_gazebo.xacro (robot description, xacro)
@@ -81,5 +81,5 @@
       <plugin name="cliff_msg_publisher" filename="libcliff_msg_publisher.so">
         <updateRate>10</updateRate>
-        <robotNumber>${robot_number}</robotNumber>
+        <robotNumber>${robot_name}</robotNumber>
       </plugin>
     </gazebo>
